Commit message: Add files via upload
Correct urdf file

File: cyton_gamma_1500.urdf (robot description, URDF)
Before this commit: robot cyton_gamma_1500, 12 links, 11 joints
Links:
- removed link base_footprint
- added link world; visual sphere radius=0.001
Joints:
- joint base_joint: parent base_footprint -> world
- joint elbow_pitch_joint: limit lower=-1.8326 upper=1.8326 effort=100.0 velocity=1.0 -> lower=-3.14159 upper=3.14159 effort=100.0 velocity=1.0
- joint elbow_yaw_joint: limit lower=-1.8326 upper=1.8326 effort=100.0 velocity=1.0 -> lower=-3.14159 upper=3.14159 effort=100.0 velocity=1.0
- joint shoulder_pitch_joint: limit lower=-1.8326 upper=1.8326 effort=100.0 velocity=1.0 -> lower=-3.14159 upper=3.14159 effort=100.0 velocity=1.0
- joint shoulder_roll_joint: limit lower=-2.618 upper=2.618 effort=100.0 velocity=1.0 -> lower=-3.14159 upper=3.14159 effort=100.0 velocity=1.0
- joint shoulder_yaw_joint: limit lower=-1.8326 upper=1.8326 effort=100.0 velocity=1.0 -> lower=-3.14159 upper=3.14159 effort=100.0 velocity=1.0
- joint wrist_pitch_joint: limit lower=-1.8326 upper=1.8326 effort=100.0 velocity=1.0 -> lower=-3.14159 upper=3.14159 effort=100.0 velocity=1.0
- joint wrist_roll_joint: limit lower=-2.61799 upper=2.61799 effort=100.0 velocity=1.0 -> lower=-3.14159 upper=3.14159 effort=100.0 velocity=1.0

Commit message: URDF update

File: cyton_gamma_1500.urdf (robot description, URDF)
Before this commit: robot cyton_gamma_1500, 12 links, 11 joints
Links:
- added link bat; visual cylinder length=0.2 radius=0.01
- added link tip
Joints:
- added joint bat_joint: type fixed, parent virtual_endeffector, child bat, origin xyz=0 0 0 rpy=0 0 0
- added joint tipshift: type fixed, parent bat, child tip, origin xyz=0 0.2 0 rpy=0 0 0

Commit message: updated urdf

File: cyton_gamma_1500.urdf (robot description, URDF)
Before this commit: robot cyton_gamma_1500, 14 links, 13 joints
Joints:
- joint tipshift: origin xyz=0 0.2 0 rpy=0 0 0 -> xyz=0.007071067812 0.15 0.007071067812 rpy=0 0 0
